File: schematic-old/espway.sch (KiCad schematic (older format))
At the start: 18 parts, among them M1 motor, M2 motor, U1 WS2812B, U2 AMS1117-5.0, U3 GY-521, U4 WS2812B, U5 WEMOS D1 mini, U6 L293D

Commit message: Updates to README and schematics
Parts:
- U2: symbol LM1117-5.0 -> LM1117-5.0-RESCUE-espway
Connections:
- new net: U3.~ (XDA), U5.~ (TX) (x3)
- new net: U1.~ (VSS), U4.~ (VSS)
- new net: U5.~ (TX), U6.~ (VCC2)
- new net: R3.1, U5.~ (TX), U6.~ (VCC2)
- new net: C7.1, M2.~, U6.~ (VCC2)
- no-connect marks 1 -> 2
Changed lines of the file:
@@
 EESchema Schematic File Version 2
+LIBS:espway-rescue
 LIBS:power
 LIBS:device
@@
 $EndComp
 $Comp
-L LM1117-5.0 U2
+L LM1117-5.0-RESCUE-espway U2
 U 1 1 58963CBC
 P 2000 1350
@@
 L GND #PWR4
 U 1 1 58964410
-P 2800 3700
-F 0 "#PWR4" H 2800 3450 50  0001 C CNN
-F 1 "GND" H 2800 3550 50  0000 C CNN
-F 2 "" H 2800 3700 50  0000 C CNN
-F 3 "" H 2800 3700 50  0000 C CNN
-	1    2800 3700
-	1    0    0    -1
+P 2650 3400
+F 0 "#PWR4" H 2650 3150 50  0001 C CNN
+F 1 "GND" H 2650 3250 50  0000 C CNN
+F 2 "" H 2650 3400 50  0000 C CNN
+F 3 "" H 2650 3400 50  0000 C CNN
+	1    2650 3400
+	0    -1   -1   0
 $EndComp
 $Comp
@@
 	1    0    0    -1
 $EndComp
-NoConn ~ 2800 2950
 $Comp
 L R R2
@@
 	6200 2200 7450 2200
 Wire Wire Line
-	2300 1350 2800 1350
-Wire Wire Line
-	2450 1350 3350 1350
+	2300 1350 3350 1350
 Wire Wire Line
 	1100 1800 2800 1800
@@
 	7900 2600 7900 2800
 Wire Wire Line
-	8650 2600 7900 2600
-Wire Wire Line
-	8650 2700 8650 2600
+	7900 2600 8650 2600
+Wire Wire Line
+	8650 2600 8650 2700
 Wire Wire Line
 	7550 3100 7450 3100
@@
 Wire Wire Line
 	6200 2500 6200 2200
-Wire Wire Line
-	3350 2950 2650 2950
-Wire Wire Line
-	3350 3100 3350 2950
-Wire Wire Line
-	3500 3100 3350 3100
-Wire Wire Line
-	2800 3250 3500 3250
-Wire Wire Line
-	2800 2800 2800 3250
-Wire Wire Line
-	2650 2800 2800 2800
 Connection ~ 3350 1350
 Connection ~ 3350 2500
@@
 	1100 1350 1700 1350
 Wire Wire Line
-	2800 3400 2800 3700
-Wire Wire Line
-	2650 3400 2800 3400
-Wire Wire Line
 	3300 4400 3150 4400
 Wire Wire Line
@@
 Connection ~ 2800 2650
 Connection ~ 2800 1800
+Wire Wire Line
+	2650 2950 3500 2950
+Wire Wire Line
+	2900 3100 3500 3100
+Wire Wire Line
+	2650 2800 3000 2800
+Wire Wire Line
+	3000 2800 3000 3250
+Wire Wire Line
+	3000 3250 3500 3250
+NoConn ~ 3000 2950
+Wire Wire Line
+	2650 3550 2900 3550
+Wire Wire Line
+	2900 3550 2900 3100
+NoConn ~ 3000 3100
 $EndSCHEMATC
